File: hardware/data_rev1/white_led.kicad_sch (KiCad schematic)
At the start: 82 parts, among them U2 IS31FL3236-TQ, U3 IS31FL3236-TQ

Commit message: Initial layout and circuit
Parts:
- C5: renamed from C1; footprint (none) -> Capacitor_SMD:C_0603_1608Metric
- C6: renamed from C3; footprint (none) -> Capacitor_SMD:C_0603_1608Metric
- C7: renamed from C2; footprint (none) -> Capacitor_SMD:C_0603_1608Metric
- C8: renamed from C4; footprint (none) -> Capacitor_SMD:C_0603_1608Metric
- D10: renamed from D13; footprint (none) -> Diode_SMD:D_0805_2012Metric
- D11: renamed from D14; footprint (none) -> Diode_SMD:D_0805_2012Metric
- D12: renamed from D15; footprint (none) -> Diode_SMD:D_0805_2012Metric
- D13: renamed from D16; footprint (none) -> Diode_SMD:D_0805_2012Metric
- D14: renamed from D17; footprint (none) -> Diode_SMD:D_0805_2012Metric
- D15: renamed from D18; footprint (none) -> Diode_SMD:D_0805_2012Metric
- D16: renamed from D25; footprint (none) -> Diode_SMD:D_0805_2012Metric
- D17: renamed from D26; footprint (none) -> Diode_SMD:D_0805_2012Metric
- D18: renamed from D27; footprint (none) -> Diode_SMD:D_0805_2012Metric
- D19: renamed from D28; footprint (none) -> Diode_SMD:D_0805_2012Metric
- D20: renamed from D29; footprint (none) -> Diode_SMD:D_0805_2012Metric
- D21: renamed from D30; footprint (none) -> Diode_SMD:D_0805_2012Metric
- D22: renamed from D37; footprint (none) -> Diode_SMD:D_0805_2012Metric
- D23: renamed from D38; footprint (none) -> Diode_SMD:D_0805_2012Metric
- D24: renamed from D39; footprint (none) -> Diode_SMD:D_0805_2012Metric
- D25: renamed from D40; footprint (none) -> Diode_SMD:D_0805_2012Metric
- D26: renamed from D41; footprint (none) -> Diode_SMD:D_0805_2012Metric
- D27: renamed from D42; footprint (none) -> Diode_SMD:D_0805_2012Metric
- D28: renamed from D43; footprint (none) -> Diode_SMD:D_0805_2012Metric
- D29: renamed from D44; footprint (none) -> Diode_SMD:D_0805_2012Metric
- D30: renamed from D45; footprint (none) -> Diode_SMD:D_0805_2012Metric
- D31: renamed from D46; footprint (none) -> Diode_SMD:D_0805_2012Metric
- D32: renamed from D47; footprint (none) -> Diode_SMD:D_0805_2012Metric
- D33: renamed from D48; footprint (none) -> Diode_SMD:D_0805_2012Metric
- D34: renamed from D49; footprint (none) -> Diode_SMD:D_0805_2012Metric
- D35: renamed from D50; footprint (none) -> Diode_SMD:D_0805_2012Metric
- D36: renamed from D51; footprint (none) -> Diode_SMD:D_0805_2012Metric
- D37: renamed from D52; footprint (none) -> Diode_SMD:D_0805_2012Metric
- D38: renamed from D53; footprint (none) -> Diode_SMD:D_0805_2012Metric
- D39: renamed from D54; footprint (none) -> Diode_SMD:D_0805_2012Metric
- D4: renamed from D1; footprint (none) -> Diode_SMD:D_0805_2012Metric
- D40: renamed from D2; footprint (none) -> Diode_SMD:D_1206_3216Metric
- D41: renamed from D4; footprint (none) -> Diode_SMD:D_1206_3216Metric
- D42: renamed from D7; footprint (none) -> Diode_SMD:D_1206_3216Metric
- D43: renamed from D8; footprint (none) -> Diode_SMD:D_1206_3216Metric
- D44: renamed from D11; footprint (none) -> Diode_SMD:D_1206_3216Metric
- D45: renamed from D12; footprint (none) -> Diode_SMD:D_1206_3216Metric
- D46: renamed from D19; footprint (none) -> Diode_SMD:D_1206_3216Metric
- D47: renamed from D20; footprint (none) -> Diode_SMD:D_1206_3216Metric
- D48: renamed from D21; footprint (none) -> Diode_SMD:D_1206_3216Metric
- D49: renamed from D22; footprint (none) -> Diode_SMD:D_1206_3216Metric
- D5: renamed from D3; footprint (none) -> Diode_SMD:D_0805_2012Metric
- D50: renamed from D23; footprint (none) -> Diode_SMD:D_1206_3216Metric
- D51: renamed from D24; footprint (none) -> Diode_SMD:D_1206_3216Metric
- D52: renamed from D31; footprint (none) -> Diode_SMD:D_1206_3216Metric
- D53: renamed from D32; footprint (none) -> Diode_SMD:D_1206_3216Metric
- D54: renamed from D33; footprint (none) -> Diode_SMD:D_1206_3216Metric
- D55: renamed from D34; footprint (none) -> Diode_SMD:D_1206_3216Metric
- D56: renamed from D35; footprint (none) -> Diode_SMD:D_1206_3216Metric
- D57: renamed from D36; footprint (none) -> Diode_SMD:D_1206_3216Metric
- D58: renamed from D55; footprint (none) -> Diode_SMD:D_1206_3216Metric
- D59: renamed from D56; footprint (none) -> Diode_SMD:D_1206_3216Metric
- D6: renamed from D5; footprint (none) -> Diode_SMD:D_0805_2012Metric
- D60: renamed from D57; footprint (none) -> Diode_SMD:D_1206_3216Metric
- D61: renamed from D58; footprint (none) -> Diode_SMD:D_1206_3216Metric
- D62: renamed from D59; footprint (none) -> Diode_SMD:D_1206_3216Metric
- D63: renamed from D60; footprint (none) -> Diode_SMD:D_1206_3216Metric
- D64: renamed from D61; footprint (none) -> Diode_SMD:D_1206_3216Metric
- D65: renamed from D62; footprint (none) -> Diode_SMD:D_1206_3216Metric
- D66: renamed from D63; footprint (none) -> Diode_SMD:D_1206_3216Metric
- D67: renamed from D64; footprint (none) -> Diode_SMD:D_1206_3216Metric
- D68: renamed from D65; footprint (none) -> Diode_SMD:D_1206_3216Metric
- D69: renamed from D66; footprint (none) -> Diode_SMD:D_1206_3216Metric
- D7: renamed from D6; footprint (none) -> Diode_SMD:D_0805_2012Metric
- D70: renamed from D67; footprint (none) -> Diode_SMD:D_1206_3216Metric
- D71: renamed from D68; footprint (none) -> Diode_SMD:D_1206_3216Metric
- D72: renamed from D69; footprint (none) -> Diode_SMD:D_1206_3216Metric
- D73: renamed from D70; footprint (none) -> Diode_SMD:D_1206_3216Metric
- D74: renamed from D71; footprint (none) -> Diode_SMD:D_1206_3216Metric
- D75: renamed from D72; footprint (none) -> Diode_SMD:D_1206_3216Metric
- D8: renamed from D9; footprint (none) -> Diode_SMD:D_0805_2012Metric
- D9: renamed from D10; footprint (none) -> Diode_SMD:D_0805_2012Metric
- R10: renamed from R2; footprint (none) -> Resistor_SMD:R_0603_1608Metric
- R11: renamed from R1; value 2k -> 5k8; footprint (none) -> Resistor_SMD:R_0603_1608Metric
- R12: renamed from R3; footprint (none) -> Resistor_SMD:R_0603_1608Metric
- R13: renamed from R4; value 2k -> 5k8; footprint (none) -> Resistor_SMD:R_0603_1608Metric
- renumbered U2 to U3, U3 to U4
Connections:
- net ~{SHTDN} renamed ~{SHTDN}_{1}
- net ~{SHTDN}_{1}: no longer R12.1, U4.39 (~{SDB})
- new net ~{SHTDN}_{2}: R12.1, U4.39 (~{SDB})
Other:
- note added: "R_{SET} = 46.8 / I_{OUT} I_{OUT} = 8 mA"
- note removed: "R_{SET} = 46.8 / I_{OUT}"
- moved on the sheet: C6, C8, D22, D23, D24, D25, D26, D27, D28, D29, D30, D31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

Commit message: Upped the IC revision for the LED driver to IS31FL3236*A*
Parts:
- U3, U4: value IS31FL3236-TQ -> IS31FL3236A-TQ
Changed lines of the file:
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@@
       (effects (font (size 1.27 1.27)) (justify left))
     )
-    (property "Value" "IS31FL3236-TQ" (at 87.2841 49.53 0)
+    (property "Value" "IS31FL3236A-TQ" (at 87.2841 49.53 0)
       (effects (font (size 1.27 1.27)) (justify left))
     )
@@
       (effects (font (size 1.27 1.27)) (justify left))
     )
-    (property "Value" "IS31FL3236-TQ" (at 204.1241 49.53 0)
+    (property "Value" "IS31FL3236A-TQ" (at 204.1241 49.53 0)
       (effects (font (size 1.27 1.27)) (justify left))
     )

Commit message: Finalized BOM
Parts:
- R10, R12: value 100k -> 51k
- R11, R13: value 5k8 -> 5k9
Changed lines of the file:
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@@
   (title_block
     (title "White LED Driving")
-    (date "2024-02-15")
-    (rev "0.1")
+    (date "2024-02-19")
+    (rev "0.2")
     (company "Savo Bajic")
   )
@@
       (effects (font (size 1.27 1.27)) (justify right))
     )
-    (property "Value" "100k" (at 60.96 71.12 0)
+    (property "Value" "51k" (at 60.96 71.12 0)
       (effects (font (size 1.27 1.27)) (justify right))
     )
@@
       (effects (font (size 1.27 1.27)) (justify left))
     )
-    (property "Value" "5k8" (at 60.96 149.86 0)
+    (property "Value" "5k9" (at 60.96 149.86 0)
       (effects (font (size 1.27 1.27)) (justify left))
     )
@@
       (effects (font (size 1.27 1.27)) (justify right))
     )
-    (property "Value" "100k" (at 177.8 71.12 0)
+    (property "Value" "51k" (at 177.8 71.12 0)
       (effects (font (size 1.27 1.27)) (justify right))
     )
@@
       (effects (font (size 1.27 1.27)) (justify left))
     )
-    (property "Value" "5k8" (at 177.8 149.86 0)
+    (property "Value" "5k9" (at 177.8 149.86 0)
       (effects (font (size 1.27 1.27)) (justify left))
     )
