File: hardware/data_rev1/white_led.kicad_sch (KiCad schematic)
At the start: 82 parts, among them U3 IS31FL3236A-TQ, U4 IS31FL3236A-TQ

Commit message: Moved to KiCad 8.0.0
Also added value for right angle LEDs toi be seperate of the head on ones
Parts:
- D40, D41, D42, D43, D44, D45, D46, D47, D48, D49, D50, D51, D52, D53, D54, D55, D56, D57, D58, D59, D60, D61, D62, D63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: value LED -> LED_RA
