File: hardware/data_rev1/data_rev1.kicad_pcb (KiCad board)
At the start: 2 copper layers, 298.7 x 69.4 mm, 4 parts, among them J1 BOARD, U1 Pico

Commit message: Initial layout and circuit
Parts:
- added C1: 0u1, Capacitor_SMD:C_0603_1608Metric, B.Cu at (84.2, 125.8)
- added C2: 10u, Resistor_SMD:R_0805_2012Metric, B.Cu at (89.5, 136.0)
- added C3: 10u, Resistor_SMD:R_0805_2012Metric, B.Cu at (97.0, 136.0)
- added C4: 1u, Capacitor_SMD:C_0603_1608Metric, B.Cu at (85.8, 125.8)
- added C5: 0u1, Capacitor_SMD:C_0603_1608Metric, B.Cu at (136.0, 114.8)
- added C6: 0u1, Capacitor_SMD:C_0603_1608Metric, B.Cu at (136.0, 137.2)
- added C7: 1u, Capacitor_SMD:C_0603_1608Metric, B.Cu at (136.0, 113.2)
- added C8: 1u, Capacitor_SMD:C_0603_1608Metric, B.Cu at (136.0, 138.8)
- added D1: STAT, LED_SMD:LED_0805_2012Metric, B.Cu at (121.5, 136.7)
- added D10: LED, Diode_SMD:D_0805_2012Metric, B.Cu at (170.0, 92.0)
- added D11: LED, Diode_SMD:D_0805_2012Metric, B.Cu at (190.0, 94.0)
- added D12: LED, Diode_SMD:D_0805_2012Metric, B.Cu at (210.0, 92.0)
- added D13: LED, Diode_SMD:D_0805_2012Metric, B.Cu at (230.1, 92.0)
- added D14: LED, Diode_SMD:D_0805_2012Metric, B.Cu at (250.0, 92.0)
- added D15: LED, Diode_SMD:D_0805_2012Metric, B.Cu at (270.0, 92.0)
- added D16: LED, Diode_SMD:D_0805_2012Metric, B.Cu at (289.0, 92.0)
- added D17: LED, Diode_SMD:D_0805_2012Metric, B.Cu at (310.0, 92.0)
- added D18: LED, Diode_SMD:D_0805_2012Metric, B.Cu at (328.5, 92.0)
- added D19: LED, Diode_SMD:D_0805_2012Metric, B.Cu at (339.0, 92.5)
- added D2: STAT, LED_SMD:LED_0805_2012Metric, B.Cu at (119.2, 136.7)
- added D20: LED, Diode_SMD:D_0805_2012Metric, B.Cu at (343.0, 105.0)
- added D21: LED, Diode_SMD:D_0805_2012Metric, B.Cu at (347.0, 122.0)
- added D22: LED, Diode_SMD:D_0805_2012Metric, B.Cu at (350.0, 139.0)
- added D23: LED, Diode_SMD:D_0805_2012Metric, B.Cu at (350.0, 152.0)
- added D24: LED, Diode_SMD:D_0805_2012Metric, B.Cu at (330.0, 152.0)
- added D25: LED, Diode_SMD:D_0805_2012Metric, B.Cu at (310.0, 143.0)
- added D26: LED, Diode_SMD:D_0805_2012Metric, B.Cu at (290.0, 152.0)
- added D27: LED, Diode_SMD:D_0805_2012Metric, B.Cu at (270.0, 152.0)
- added D28: LED, Diode_SMD:D_0805_2012Metric, B.Cu at (250.0, 152.0)
- added D29: LED, Diode_SMD:D_0805_2012Metric, B.Cu at (230.0, 152.0)
- added D3: STAT, LED_SMD:LED_0805_2012Metric, B.Cu at (117.0, 136.7)
- added D30: LED, Diode_SMD:D_0805_2012Metric, B.Cu at (210.0, 142.0)
- added D31: LED, Diode_SMD:D_0805_2012Metric, B.Cu at (190.0, 143.0)
- added D32: LED, Diode_SMD:D_0805_2012Metric, B.Cu at (170.0, 152.0)
- added D33: LED, Diode_SMD:D_0805_2012Metric, B.Cu at (150.0, 152.0)
- added D34: LED, Diode_SMD:D_0805_2012Metric, B.Cu at (130.0, 152.0)
- added D35: LED, Diode_SMD:D_0805_2012Metric, B.Cu at (110.0, 152.0)
- added D36: LED, Diode_SMD:D_0805_2012Metric, B.Cu at (87.0, 153.5)
- added D37: LED, Diode_SMD:D_0805_2012Metric, B.Cu at (66.0, 151.5)
- added D38: LED, Diode_SMD:D_0805_2012Metric, B.Cu at (66.0, 139.0)
- added D39: LED, Diode_SMD:D_0805_2012Metric, B.Cu at (70.0, 122.0)
- added D4: LED, Diode_SMD:D_0805_2012Metric, B.Cu at (72.5, 111.0)
- added D40: LED, Diode_SMD:D_1206_3216Metric, B.Cu at (75.5, 97.0)
- added D41: LED, Diode_SMD:D_1206_3216Metric, B.Cu at (83.0, 92.0)
- added D42: LED, Diode_SMD:D_1206_3216Metric, B.Cu at (100.0, 92.0)
- added D43: LED, Diode_SMD:D_1206_3216Metric, B.Cu at (120.0, 92.0)
- added D44: LED, Diode_SMD:D_1206_3216Metric, B.Cu at (140.0, 92.0)
- added D45: LED, Diode_SMD:D_1206_3216Metric, B.Cu at (160.0, 92.0)
- added D46: LED, Diode_SMD:D_1206_3216Metric, B.Cu at (180.0, 92.0)
- added D47: LED, Diode_SMD:D_1206_3216Metric, B.Cu at (201.0, 92.0)
- added D48: LED, Diode_SMD:D_1206_3216Metric, B.Cu at (220.0, 92.0)
- added D49: LED, Diode_SMD:D_1206_3216Metric, B.Cu at (240.0, 92.0)
- added D5: LED, Diode_SMD:D_0805_2012Metric, B.Cu at (78.0, 93.0)
- added D50: LED, Diode_SMD:D_1206_3216Metric, B.Cu at (260.0, 92.0)
- added D51: LED, Diode_SMD:D_1206_3216Metric, B.Cu at (280.0, 92.0)
- added D52: LED, Diode_SMD:D_1206_3216Metric, B.Cu at (300.0, 92.0)
- added D53: LED, Diode_SMD:D_1206_3216Metric, B.Cu at (321.4, 92.0)
- added D54: LED, Diode_SMD:D_1206_3216Metric, B.Cu at (335.0, 92.0)
- added D55: LED, Diode_SMD:D_1206_3216Metric, B.Cu at (341.5, 97.0)
- added D56: LED, Diode_SMD:D_1206_3216Metric, B.Cu at (345.0, 113.5)
- added D57: LED, Diode_SMD:D_1206_3216Metric, B.Cu at (348.5, 130.0)
- added D58: LED, Diode_SMD:D_1206_3216Metric, B.Cu at (352.5, 147.0)
- added D59: LED, Diode_SMD:D_1206_3216Metric, B.Cu at (340.0, 152.0)
- added D6: LED, Diode_SMD:D_0805_2012Metric, B.Cu at (90.0, 92.0)
- added D60: LED, Diode_SMD:D_1206_3216Metric, B.Cu at (320.0, 143.0)
- added D61: LED, Diode_SMD:D_1206_3216Metric, B.Cu at (300.0, 148.0)
- added D62: LED, Diode_SMD:D_1206_3216Metric, B.Cu at (280.0, 152.0)
- added D63: LED, Diode_SMD:D_1206_3216Metric, B.Cu at (260.0, 152.0)
- added D64: LED, Diode_SMD:D_1206_3216Metric, B.Cu at (240.0, 152.0)
- added D65: LED, Diode_SMD:D_1206_3216Metric, B.Cu at (220.0, 152.0)
- added D66: LED, Diode_SMD:D_1206_3216Metric, B.Cu at (200.0, 142.0)
- added D67: LED, Diode_SMD:D_1206_3216Metric, B.Cu at (180.0, 148.0)
- added D68: LED, Diode_SMD:D_1206_3216Metric, B.Cu at (160.0, 152.0)
- added D69: LED, Diode_SMD:D_1206_3216Metric, B.Cu at (140.0, 152.0)
- added D7: LED, Diode_SMD:D_0805_2012Metric, B.Cu at (110.0, 92.0)
- added D70: LED, Diode_SMD:D_1206_3216Metric, B.Cu at (120.0, 152.0)
- added D71: LED, Diode_SMD:D_1206_3216Metric, B.Cu at (100.0, 152.0)
- added D72: LED, Diode_SMD:D_1206_3216Metric, B.Cu at (72.0, 152.0)
- added D73: LED, Diode_SMD:D_1206_3216Metric, B.Cu at (64.0, 147.0)
- added D74: LED, Diode_SMD:D_1206_3216Metric, B.Cu at (68.0, 130.0)
- added D75: LED, Diode_SMD:D_1206_3216Metric, B.Cu at (72.0, 115.0)
- added D8: LED, Diode_SMD:D_0805_2012Metric, B.Cu at (130.0, 92.0)
- added D9: LED, Diode_SMD:D_0805_2012Metric, B.Cu at (150.0, 92.0)
- added G***: LOGO, logo:tainy, B.Cu at (254.5, 140.0)
- added J1: AudioJack3, Connector_Audio:Jack_3.5mm_CUI_SJ-3523-SMT_Horizontal, B.Cu at (81.0, 147.0)
- added J2: AudioJack3, Connector_Audio:Jack_3.5mm_CUI_SJ-3523-SMT_Horizontal, B.Cu at (93.2, 147.0)
- added R1: 51k, Resistor_SMD:R_0603_1608Metric, B.Cu at (87.5, 136.0)
- added R10: 100k, Resistor_SMD:R_0603_1608Metric, B.Cu at (136.0, 116.2)
- added R11: 5k8, Resistor_SMD:R_0603_1608Metric, B.Cu at (136.0, 111.8)
- added R12: 100k, Resistor_SMD:R_0603_1608Metric, B.Cu at (136.0, 140.2)
- added R13: 5k8, Resistor_SMD:R_0603_1608Metric, B.Cu at (136.0, 135.8)
- added R2: 51k, Resistor_SMD:R_0603_1608Metric, B.Cu at (91.5, 136.0)
- added R3: 51k, Resistor_SMD:R_0603_1608Metric, B.Cu at (99.0, 136.0)
- added R4: 51k, Resistor_SMD:R_0603_1608Metric, B.Cu at (95.0, 136.0)
- added R5: 5k1, Resistor_SMD:R_0603_1608Metric, B.Cu at (88.8, 125.8)
- added R6: 5k1, Resistor_SMD:R_0603_1608Metric, B.Cu at (87.2, 125.8)
- added R7: 130, Resistor_SMD:R_0603_1608Metric, B.Cu at (121.5, 140.2)
- added R8: 130, Resistor_SMD:R_0603_1608Metric, B.Cu at (119.2, 140.2)
- added R9: 130, Resistor_SMD:R_0603_1608Metric, B.Cu at (117.0, 140.2)
- added SW1: PTS636, Button_Switch_SMD:SW_SPST_CK_RS282G05A3, B.Cu at (113.0, 137.0)
- added SW2: PTS636, Button_Switch_SMD:SW_SPST_CK_RS282G05A3, B.Cu at (108.0, 137.0)
- added SW3: PTS636, Button_Switch_SMD:SW_SPST_CK_RS282G05A3, B.Cu at (103.0, 137.0)
- added U1: CAP1206-x-AIA, Package_DFN_QFN:DFN-10-1EP_3x3mm_P0.5mm_EP1.55x2.48mm, B.Cu at (79.6, 125.4)
- added U3: IS31FL3236-TQ, Package_QFP:TQFP-48-1EP_7x7mm_P0.5mm_EP4.11x4.11mm, B.Cu at (143.8, 112.8)
- added U4: IS31FL3236-TQ, Package_QFP:TQFP-48-1EP_7x7mm_P0.5mm_EP4.11x4.11mm, B.Cu at (143.8, 137.0)
- moved U2 17.7 mm to (102.3, 112.4)
- renumbered J1 to J3, U1 to U2
Connections:
- J3 pad 1: unconnected-(J1-Pin_1-Pad1) -> /PAD_{0}
- J3 pad 2: unconnected-(J1-Pin_2-Pad2) -> /PAD_{1}
- J3 pad 3: unconnected-(J1-Pin_3-Pad3) -> /PAD_{2}
- J3 pad 4: unconnected-(J1-Pin_4-Pad4) -> /PAD_{3}
- J3 pad 5: unconnected-(J1-Pin_5-Pad5) -> /PAD_{DA}
- J3 pad 6: unconnected-(J1-Pin_6-Pad6) -> /PAD_{TA}
- U2 pad 1: unconnected-(U1-GPIO0-Pad1) -> /SDA
- U2 pad 13: unconnected-(U1-GND-Pad13) -> GND
- U2 pad 18: unconnected-(U1-GND-Pad18) -> GND
- U2 pad 2: unconnected-(U1-GPIO1-Pad2) -> /SCL
- U2 pad 20: unconnected-(U1-GPIO15-Pad20) -> /~{SHTDN}_{1}
- U2 pad 21: unconnected-(U1-GPIO16-Pad21) -> /~{SHTDN}_{2}
- U2 pad 22: unconnected-(U1-GPIO17-Pad22) -> /LED_{1}
- U2 pad 23: unconnected-(U1-GND-Pad23) -> GND
- U2 pad 24: unconnected-(U1-GPIO18-Pad24) -> /LED_{2}
- U2 pad 25: unconnected-(U1-GPIO19-Pad25) -> /LED_{3}
- U2 pad 26: unconnected-(U1-GPIO20-Pad26) -> /BUT_{1}
- U2 pad 27: unconnected-(U1-GPIO21-Pad27) -> /BUT_{2}
- U2 pad 28: unconnected-(U1-GND-Pad28) -> GND
- U2 pad 3: unconnected-(U1-GND-Pad3) -> GND
- U2 pad 30: unconnected-(U1-RUN-Pad30) -> /RUN
- U2 pad 31: unconnected-(U1-GPIO26_ADC0-Pad31) -> /RIGHT
- U2 pad 32: unconnected-(U1-GPIO27_ADC1-Pad32) -> /LEFT
- U2 pad 33: unconnected-(U1-AGND-Pad33) -> GND
- U2 pad 36: unconnected-(U1-3V3-Pad36) -> +3V3
- U2 pad 38: unconnected-(U1-GND-Pad38) -> GND
- U2 pad 42: unconnected-(U1-GND-Pad42) -> GND
- U2 pad 8: unconnected-(U1-GND-Pad8) -> GND
Routing:
- net /PAD_{TA}: track 0.00 -> 298.8 mm, vias 0 -> 1
- net Net-(D58-K): track 0.00 -> 227.0 mm
- net Net-(D23-K): track 0.00 -> 226.7 mm
- net Net-(D22-K): track 0.00 -> 224.1 mm
- net Net-(D57-K): track 0.00 -> 217.8 mm
- net Net-(D59-K): track 0.00 -> 214.7 mm
- net Net-(D55-K): track 0.00 -> 212.0 mm
- net Net-(D21-K): track 0.00 -> 211.9 mm
- net Net-(D20-K): track 0.00 -> 211.4 mm
- net Net-(D56-K): track 0.00 -> 210.5 mm
- net Net-(D19-K): track 0.00 -> 210.5 mm
- net Net-(D24-K): track 0.00 -> 208.8 mm
- net Net-(D54-K): track 0.00 -> 207.6 mm
- net Net-(D18-K): track 0.00 -> 199.8 mm
- net Net-(D53-K): track 0.00 -> 192.3 mm
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- added copper zone on B.Cu, net +3V3
- added copper zone on B.Cu, net GND
Other:
- board text added: "0xCAB0"

Commit message: Moved audio jacks to the side. Ordered.
Parts:
- moved J2 29.0 mm to (75.0, 124.5), turned to -90 degrees
- moved R3 20.6 mm to (83.0, 149.0), turned to 0 degrees
- moved C3 17.8 mm to (83.0, 147.0), turned to 180 degrees
- moved R4 15.0 mm to (83.0, 145.0), turned to 180 degrees
- moved J1 12.4 mm to (72.0, 138.5), turned to -90 degrees
- moved R2 11.0 mm to (83.0, 143.0), turned to 180 degrees
- moved U1 8.77 mm to (84.9, 132.4), turned to -90 degrees
- moved C2 8.20 mm to (83.0, 141.0), turned to 180 degrees
- moved D38 7.91 mm to (68.5, 131.5), turned to 180 degrees
- moved R1 5.41 mm to (83.0, 139.0), turned to 0 degrees
- moved U2 5.03 mm to (97.5, 111.0)
- moved D39 4.72 mm to (74.0, 119.5)
- moved D75 4.61 mm to (68.5, 118.0)
- moved R5 4.12 mm to (85.5, 123.2), turned to 180 degrees
- moved D4 3.31 mm to (69.2, 111.6), turned to -105 degrees
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Connections:
- U1 pad 10: /PAD_{1} -> /PAD_{0}
- U1 pad 9: /PAD_{0} -> /PAD_{1}
- U2 pad 1: /SDA -> unconnected-(U2-GPIO0-Pad1)
- U2 pad 16: unconnected-(U2-GPIO12-Pad16) -> /SDA
- U2 pad 17: unconnected-(U2-GPIO13-Pad17) -> /SCL
- U2 pad 2: /SCL -> unconnected-(U2-GPIO1-Pad2)
Routing:
- net /PAD_{1}: track 19.9 -> 62.0 mm
- net /PAD_{3}: track 49.4 -> 13.3 mm
- net /SCL: track 150.6 -> 118.5 mm, vias 4 -> 5
- net /PAD_{0}: track 52.2 -> 83.5 mm
- net /SDA: track 150.5 -> 121.5 mm, vias 4 -> 3
- net GND: track 36.8 -> 15.2 mm, vias 2 -> 0
- net /PAD_{DA}: track 85.1 -> 68.9 mm
- net +3V3: track 119.1 -> 134.8 mm
- net /RIGHT: track 18.7 -> 34.3 mm
- net /PAD_{TA}: track 298.8 -> 285.4 mm
- net /LEFT: track 21.3 -> 32.5 mm
- net Net-(D38-K): track 78.5 -> 88.5 mm
- net /LEFT_{RAW}: track 16.5 -> 23.8 mm, vias 0 -> 2
- net Net-(D75-K): track 90.9 -> 96.4 mm
- net /PAD_{2}: track 13.3 -> 8.09 mm
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Other:
- board text added: "0xCAB0 - Rev. ${REVISION}"
- board text removed: "0xCAB0"

Commit message: Upped the IC revision for the LED driver to IS31FL3236*A*
Parts:
- U3, U4: value IS31FL3236-TQ -> IS31FL3236A-TQ
Changed lines of the file:
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@@
         (effects (font (size 1 1) (thickness 0.15)) (justify mirror))
     )
-    (fp_text value "IS31FL3236-TQ" (at 0 -5.85 90) (layer "B.Fab")
+    (fp_text value "IS31FL3236A-TQ" (at 0 -5.85 90) (layer "B.Fab")
         (effects (font (size 1 1) (thickness 0.15)) (justify mirror))
     )
@@
         (effects (font (size 1 1) (thickness 0.15)) (justify mirror))
     )
-    (fp_text value "IS31FL3236-TQ" (at 0 -5.85 90) (layer "B.Fab")
+    (fp_text value "IS31FL3236A-TQ" (at 0 -5.85 90) (layer "B.Fab")
         (effects (font (size 1 1) (thickness 0.15)) (justify mirror))
     )

Commit message: Finalized BOM
Parts:
- R10, R12: value 100k -> 51k
- R11, R13: value 5k8 -> 5k9
- R5, R6: value 5k1 -> 5k9
Changed lines of the file:
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@@
         (effects (font (size 1 1) (thickness 0.15)) (justify mirror))
     )
-    (fp_text value "100k" (at 0 -1.43) (layer "B.Fab")
+    (fp_text value "51k" (at 0 -1.43) (layer "B.Fab")
         (effects (font (size 1 1) (thickness 0.15)) (justify mirror))
     )
@@
         (effects (font (size 1 1) (thickness 0.15)) (justify mirror))
     )
-    (fp_text value "5k1" (at 0 -1.43) (layer "B.Fab")
+    (fp_text value "5k9" (at 0 -1.43) (layer "B.Fab")
         (effects (font (size 1 1) (thickness 0.15)) (justify mirror))
     )
@@
         (effects (font (size 1 1) (thickness 0.15)) (justify mirror))
     )
-    (fp_text value "5k8" (at 0 -1.43) (layer "B.Fab")
+    (fp_text value "5k9" (at 0 -1.43) (layer "B.Fab")
         (effects (font (size 1 1) (thickness 0.15)) (justify mirror))
     )
@@
         (effects (font (size 1 1) (thickness 0.15)) (justify mirror))
     )
-    (fp_text value "5k1" (at 0 -1.43) (layer "B.Fab")
+    (fp_text value "5k9" (at 0 -1.43) (layer "B.Fab")
         (effects (font (size 1 1) (thickness 0.15)) (justify mirror))
     )
@@
         (effects (font (size 1 1) (thickness 0.15)) (justify mirror))
     )
-    (fp_text value "5k8" (at 0 -1.43) (layer "B.Fab")
+    (fp_text value "5k9" (at 0 -1.43) (layer "B.Fab")
         (effects (font (size 1 1) (thickness 0.15)) (justify mirror))
     )
@@
         (effects (font (size 1 1) (thickness 0.15)) (justify mirror))
     )
-    (fp_text value "100k" (at 0 -1.43) (layer "B.Fab")
+    (fp_text value "51k" (at 0 -1.43) (layer "B.Fab")
         (effects (font (size 1 1) (thickness 0.15)) (justify mirror))
     )

Commit message: Added labels for LED lines
Connections:
- net Net-(D10-K) renamed /White LED/D0.12
- net Net-(D11-K) renamed /White LED/D0.14
- net Net-(D12-K) renamed /White LED/D0.16
- net Net-(D13-K) renamed /White LED/D0.18
- net Net-(D14-K) renamed /White LED/D0.20
- net Net-(D15-K) renamed /White LED/D0.22
- net Net-(D16-K) renamed /White LED/D0.24
- net Net-(D17-K) renamed /White LED/D0.26
- net Net-(D18-K) renamed /White LED/D0.28
- net Net-(D19-K) renamed /White LED/D0.30
- net Net-(D20-K) renamed /White LED/D0.32
- net Net-(D21-K) renamed /White LED/D0.34
- net Net-(D22-K) renamed /White LED/D1.00
- net Net-(D23-K) renamed /White LED/D1.02
- net Net-(D24-K) renamed /White LED/D1.04
- net Net-(D25-K) renamed /White LED/D1.06
- net Net-(D26-K) renamed /White LED/D1.08
- net Net-(D27-K) renamed /White LED/D1.10
- net Net-(D28-K) renamed /White LED/D1.12
- net Net-(D29-K) renamed /White LED/D1.14
- net Net-(D30-K) renamed /White LED/D1.16
- net Net-(D31-K) renamed /White LED/D1.18
- net Net-(D32-K) renamed /White LED/D1.20
- net Net-(D33-K) renamed /White LED/D1.22
- net Net-(D34-K) renamed /White LED/D1.24
- net Net-(D35-K) renamed /White LED/D1.26
- net Net-(D36-K) renamed /White LED/D1.28
- net Net-(D37-K) renamed /White LED/D1.30
- net Net-(D38-K) renamed /White LED/D1.32
- net Net-(D39-K) renamed /White LED/D1.34
- net Net-(D4-K) renamed /White LED/D0.00
- net Net-(D40-K) renamed /White LED/D0.01
- net Net-(D41-K) renamed /White LED/D0.03
- net Net-(D42-K) renamed /White LED/D0.05
- net Net-(D43-K) renamed /White LED/D0.07
- net Net-(D44-K) renamed /White LED/D0.09
- net Net-(D45-K) renamed /White LED/D0.11
- net Net-(D46-K) renamed /White LED/D0.13
- net Net-(D47-K) renamed /White LED/D0.15
- net Net-(D48-K) renamed /White LED/D0.17
- net Net-(D49-K) renamed /White LED/D0.19
- net Net-(D5-K) renamed /White LED/D0.02
- net Net-(D50-K) renamed /White LED/D0.21
- net Net-(D51-K) renamed /White LED/D0.23
- net Net-(D52-K) renamed /White LED/D0.25
- net Net-(D53-K) renamed /White LED/D0.27
- net Net-(D54-K) renamed /White LED/D0.29
- net Net-(D55-K) renamed /White LED/D0.31
- net Net-(D56-K) renamed /White LED/D0.33
- net Net-(D57-K) renamed /White LED/D0.35
- net Net-(D58-K) renamed /White LED/D1.01
- net Net-(D59-K) renamed /White LED/D1.03
- net Net-(D6-K) renamed /White LED/D0.04
- net Net-(D60-K) renamed /White LED/D1.05
- net Net-(D61-K) renamed /White LED/D1.07
- net Net-(D62-K) renamed /White LED/D1.09
- net Net-(D63-K) renamed /White LED/D1.11
- net Net-(D64-K) renamed /White LED/D1.13
- net Net-(D65-K) renamed /White LED/D1.15
- net Net-(D66-K) renamed /White LED/D1.17
- net Net-(D67-K) renamed /White LED/D1.19
- net Net-(D68-K) renamed /White LED/D1.21
- net Net-(D69-K) renamed /White LED/D1.23
- net Net-(D7-K) renamed /White LED/D0.06
- net Net-(D70-K) renamed /White LED/D1.25
- net Net-(D71-K) renamed /White LED/D1.27
- net Net-(D72-K) renamed /White LED/D1.29
- net Net-(D73-K) renamed /White LED/D1.31
- net Net-(D74-K) renamed /White LED/D1.33
- net Net-(D75-K) renamed /White LED/D1.35
- net Net-(D8-K) renamed /White LED/D0.08
- net Net-(D9-K) renamed /White LED/D0.10
