File: hardware/data_rev0/data_rev0.kicad_pcb (KiCad board)
At the start: 2 copper layers, 298.7 x 69.4 mm, 107 parts, among them J1 AudioJack3, J2 AudioJack3, J3 BOARD, SW3 PTS636, U1 CAP1206-x-AIA, U2 Pico, U3 IS31FL3236A-TQ, U4 IS31FL3236A-TQ

Commit message: Added Rev 0 project
Started some of my changes on Rev 1. Also changed the RP Pico footprint to have solderpaste on the pads.
Parts:
- added SW1: PTS636, Button_Switch_SMD:SW_SPST_CK_RS282G05A3, B.Cu at (113.0, 137.0)
- added SW2: PTS636, Button_Switch_SMD:SW_SPST_CK_RS282G05A3, B.Cu at (108.0, 137.0)
Connections:
- J1 pad S: GNDA -> GND
- J2 pad S: GNDA -> GND
- R2 pad 2: GNDA -> GND
- R4 pad 2: GNDA -> GND
- U1 pad 2: /CAP_{INT} -> GND
- U2 pad 26: unconnected-(U2-GPIO20-Pad26) -> /BUT_{1}
- U2 pad 27: /CAP_{INT} -> /BUT_{2}
- U2 pad 33: GNDA -> GND
Routing:
- net GNDA: track 65.1 -> 0.00 mm
- net GND: track 0.00 -> 15.2 mm
- net /BUT_{1}: track 0.00 -> 13.4 mm
- net /BUT_{2}: track 0.00 -> 13.0 mm
Other:
- board text removed: "Move all connectors to the edge"
